File: doc/schematic/imble3_demo.kicad_sch (KiCad schematic)
At the start: 14 parts, among them J1 Conn_01x06, J2 Conn_01x09, J3 Conn_01x02, SW1 SW_Push_DPDT, SW4 SW_Push, SW5 SW_Push

Commit message: change icon
Parts:
- added R6: 1k, symbol Device:R_US
- added SW2: SW_SPDT, symbol Switch:SW_SPDT
- R1: value 3.3k -> 1k
Connections:
- net GNDREF: now also R6.2, SW2.1 (A); no longer R2.2, SW1.6 (C)
- net at SW1.2 (B): now also SW2.3 (C)
- new net: R2.2, R6.1, SW1.6 (C)

Commit message: Update for New Hardware Design
- Updated assets to reflect new hardware design. Adjusted images and other resources to match the latest specifications.
Parts:
- removed R6: 1k, symbol Device:R_US
- removed SW2: SW_SPDT, symbol Switch:SW_SPDT
- R1: value 1k -> 3.3k
Connections:
- net GNDREF: now also R2.2, SW1.6 (C)
